File: Hardware/RedBoard_Plus.brd (EAGLE design)
At the start: 68.6 x 58.4 mm, 179 parts, among them IC3 LM1117, J1 DNP, J2 ISP, J3 5.5x2.1mm Barrel, J4 QWIIC_RIGHT_ANGLE, J5 USB Female Type C Connector, Q1 20V/4.2A/52mΩ/1.4W, Q2 310mA/60V/1.6Ω, Q3 310mA/60V/1.6Ω, U1 CH340G, U3 3.3V, U4 ATMEGA328P_TQFP, Y1 16MHz, Y2 12MHz

Commit message: Update silk on bottom of board
Move "1" label more in-line with others
Add "~" to pins 10 and 11
Parts:
- removed U$74: (no value), output:100
- removed U$75: (no value), output:110
- added U$21: (no value), output:11#0
- added U$9: (no value), output:10#0
- moved U$65 0.51 mm to (61.0, 57.1)
Changed lines of the file:
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@@
 <?xml version="1.0" encoding="utf-8"?>
 <!DOCTYPE eagle SYSTEM "eagle.dtd">
-<eagle version="9.5.2">
+<eagle version="9.6.2">
 <drawing>
 <settings>
@@
 <element name="U$63" library="output" package="A70" value="" x="25.4" y="1.905" smashed="yes" rot="R90"/>
 <element name="U$64" library="output" package="00" value="" x="63.5" y="57.15" smashed="yes" rot="MR270"/>
-<element name="U$65" library="output" package="10" value="" x="60.96" y="56.642" smashed="yes" rot="MR270"/>
+<element name="U$65" library="output" package="10" value="" x="60.96" y="57.15" smashed="yes" rot="MR270"/>
 <element name="U$66" library="output" package="20" value="" x="58.42" y="57.15" smashed="yes" rot="MR270"/>
 <element name="U$67" library="output" package="3#0" value="" x="55.88" y="57.15" smashed="yes" rot="MR270"/>
@@
 <element name="U$72" library="output" package="80" value="" x="41.656" y="57.15" smashed="yes" rot="MR270"/>
 <element name="U$73" library="output" package="9#0" value="" x="39.116" y="57.15" smashed="yes" rot="MR270"/>
-<element name="U$74" library="output" package="100" value="" x="36.576" y="57.15" smashed="yes" rot="MR270"/>
-<element name="U$75" library="output" package="110" value="" x="34.036" y="57.15" smashed="yes" rot="MR270"/>
 <element name="U$76" library="output" package="120" value="" x="31.496" y="57.15" smashed="yes" rot="MR270"/>
 <element name="U$77" library="output" package="130" value="" x="28.956" y="57.15" smashed="yes" rot="MR270"/>
@@
 <element name="U$107" library="output" package="_GND_0" value="" x="43.18" y="9.525" smashed="yes" rot="MR270"/>
 <element name="LOGO1" library="SparkFun-Aesthetics" package="QWIIC_5MM" value="QWIIC_LOGO_5MM" x="61.722" y="19.05" smashed="yes" rot="R90"/>
+<element name="U$9" library="output" package="10#0" value="" x="36.576" y="57.15" smashed="yes" rot="MR270"/>
+<element name="U$21" library="output" package="11#0" value="" x="34.036" y="57.15" smashed="yes" rot="MR270"/>
 </elements>
 <signals>
