File: Hardware/Production/RedBoard_Plus-Panel.brd (EAGLE design)
At the start: 365 x 131.6 mm, 1786 parts, among them IC1 LM1117, IC10 LM1117, IC2 LM1117, IC3 LM1117, IC4 LM1117, IC5 LM1117, IC6 LM1117, IC7 LM1117, IC8 LM1117, IC9 LM1117, J1 DNP, J10 DNP, J11 ISP, J12 5.5x2.1mm Barrel, J13 QWIIC_RIGHT_ANGLE, J14 USB Female Type C Connector, J15 DNP, J16 ISP, J17 5.5x2.1mm Barrel, J18 QWIIC_RIGHT_ANGLE, J19 USB Female Type C Connector, J2 ISP, J20 DNP, J21 ISP, J22 5.5x2.1mm Barrel, J23 QWIIC_RIGHT_ANGLE, J24 USB Female Type C Connector, J25 DNP, J26 ISP, J27 5.5x2.1mm Barrel, J28 QWIIC_RIGHT_ANGLE, J29 USB Female Type C Connector, J3 5.5x2.1mm Barrel, J30 DNP, J31 ISP, J32 5.5x2.1mm Barrel, J33 QWIIC_RIGHT_ANGLE, J34 USB Female Type C Connector, J35 DNP, J36 ISP, J37 5.5x2.1mm Barrel, J38 QWIIC_RIGHT_ANGLE, J39 USB Female Type C Connector, J4 QWIIC_RIGHT_ANGLE, J40 DNP, J41 ISP, J42 5.5x2.1mm Barrel, J43 QWIIC_RIGHT_ANGLE, J44 USB Female Type C Connector, J45 DNP, J46 ISP, J47 5.5x2.1mm Barrel, J48 QWIIC_RIGHT_ANGLE, J49 USB Female Type C Connector, J5 USB Female Type C Connector, J50 DNP, J6 ISP, J7 5.5x2.1mm Barrel, J8 QWIIC_RIGHT_ANGLE, J9 USB Female Type C Connector, Q1 20V/4.2A/52mΩ/1.4W, Q10 20V/4.2A/52mΩ/1.4W, Q11 310mA/60V/1.6Ω, Q12 310mA/60V/1.6Ω, Q13 20V/4.2A/52mΩ/1.4W, Q14 310mA/60V/1.6Ω, Q15 310mA/60V/1.6Ω, Q16 20V/4.2A/52mΩ/1.4W, Q17 310mA/60V/1.6Ω, Q18 310mA/60V/1.6Ω, Q19 20V/4.2A/52mΩ/1.4W, Q2 310mA/60V/1.6Ω, Q20 310mA/60V/1.6Ω, Q21 310mA/60V/1.6Ω, Q22 20V/4.2A/52mΩ/1.4W, Q23 310mA/60V/1.6Ω, Q24 310mA/60V/1.6Ω, Q25 20V/4.2A/52mΩ/1.4W, Q26 310mA/60V/1.6Ω, Q27 310mA/60V/1.6Ω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

Commit message: Update panel
Parts:
- moved E$3 12.7 mm to (360.3, 114.7)
- moved E$4 12.7 mm to (360.3, 114.7)
- moved C136 10.2 mm to (319.9, 80.4)
- moved C137 10.2 mm to (322.1, 84.8)
- moved C139 10.2 mm to (296.7, 87.6)
- moved C141 10.2 mm to (314.5, 90.8)
- moved C142 10.2 mm to (288.3, 91.1)
- moved C143 10.2 mm to (296.7, 89.2)
- moved C144 10.2 mm to (297.2, 91.9)
- moved C61 10.2 mm to (319.9, 21.5)
- moved C62 10.2 mm to (322.1, 25.8)
- moved C64 10.2 mm to (296.7, 28.7)
- moved C66 10.2 mm to (314.5, 31.9)
- moved C67 10.2 mm to (288.3, 32.1)
- moved C68 10.2 mm to (296.7, 30.2)
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Other:
- board size 365 x 131.6 mm -> 380.2 x 131.1 mm
- board text added: "Route Out"

Commit message: Re-panelize without fiducials moved to left+right corners
Parts:
- moved E$5 16.8 mm to (9.40, -2.10)
- moved E$6 16.8 mm to (9.40, -2.10)
- moved E$1 15.3 mm to (9.40, 119.4)
- moved E$2 15.3 mm to (9.40, 119.4)
- moved E$3 8.47 mm to (353.3, 119.4)
- moved E$4 8.47 mm to (353.3, 119.4)
Changed lines of the file:
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@@
 <element name="U$979" library="output" package="10#0" value="" x="323.088" y="116.078" smashed="yes" rot="MR270"/>
 <element name="U$980" library="output" package="11#0" value="" x="320.548" y="116.078" smashed="yes" rot="MR270"/>
-<element name="E$1" library="SparkFun-Aesthetics" package="FIDUCIAL-1X2" value="" x="-5.16381875" y="114.681" smashed="yes"/>
-<element name="E$2" library="SparkFun-Aesthetics" package="FIDUCIAL-1X2" value="" x="-5.16381875" y="114.681" smashed="yes" rot="MR0"/>
-<element name="E$3" library="SparkFun-Aesthetics" package="FIDUCIAL-1X2" value="" x="360.25581875" y="114.681" smashed="yes"/>
-<element name="E$4" library="SparkFun-Aesthetics" package="FIDUCIAL-1X2" value="" x="360.25581875" y="114.681" smashed="yes" rot="MR0"/>
-<element name="E$5" library="SparkFun-Retired" package="FIDUCIAL-1.5X3" value="" x="-5.16381875" y="6.35" smashed="yes"/>
-<element name="E$6" library="SparkFun-Retired" package="FIDUCIAL-1.5X3" value="" x="-5.16381875" y="6.35" smashed="yes" rot="MR0"/>
+<element name="E$1" library="SparkFun-Aesthetics" package="FIDUCIAL-1X2" value="" x="9.398" y="119.4435" smashed="yes"/>
+<element name="E$2" library="SparkFun-Aesthetics" package="FIDUCIAL-1X2" value="" x="9.398" y="119.4435" smashed="yes" rot="MR0"/>
+<element name="E$3" library="SparkFun-Aesthetics" package="FIDUCIAL-1X2" value="" x="353.2505" y="119.4435" smashed="yes"/>
+<element name="E$4" library="SparkFun-Aesthetics" package="FIDUCIAL-1X2" value="" x="353.2505" y="119.4435" smashed="yes" rot="MR0"/>
+<element name="E$5" library="SparkFun-Retired" package="FIDUCIAL-1.5X3" value="" x="9.398" y="-2.0955" smashed="yes"/>
+<element name="E$6" library="SparkFun-Retired" package="FIDUCIAL-1.5X3" value="" x="9.398" y="-2.0955" smashed="yes" rot="MR0"/>
 </elements>
 <signals>
